Commit message: up-to-date configuration for final demo

File: mmseq_assets/scenes/urdf/restaurant.urdf (robot description, URDF)
Before this commit: robot robot, 13 links, 12 joints
Links:
- link chair_1: geometry collision mesh filename=file:///home/tracy/Project/catkin_ws/src/mm_sequential_task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; visual mesh filename=file:///home/tracy/Project/catkin_ws/src/mm_sequential_task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
- link chair_2: geometry collision mesh filename=file:///home/tracy/Project/catkin_ws/src/mm_sequential_task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; visual mesh filename=file:///home/tracy/Project/catkin_ws/src/mm_sequential_task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
- link chair_3: geometry collision mesh filename=file:///home/tracy/Project/catkin_ws/src/mm_sequential_task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; visual mesh filename=file:///home/tracy/Project/catkin_ws/src/mm_sequential_task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
- link chair_4: geometry collision mesh filename=file:///home/tracy/Project/catkin_ws/src/mm_sequential_task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; visual mesh filename=file:///home/tracy/Project/catkin_ws/src/mm_sequential_task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
- link chair_5: geometry collision mesh filename=file:///home/tracy/Project/catkin_ws/src/mm_sequential_task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; visual mesh filename=file:///home/tracy/Project/catkin_ws/src/mm_sequential_task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
- link chair_6: geometry collision mesh filename=file:///home/tracy/Project/catkin_ws/src/mm_sequential_task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; visual mesh filename=file:///home/tracy/Project/catkin_ws/src/mm_sequential_task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
Joints:
- joint chair_1_joint: origin xyz=-3. -3. 0. rpy=0 0 0 -> xyz=0 -3. 0. rpy=0 0 0
- joint chair_2_joint: origin xyz=-3. 0. 0. rpy=0 0 0 -> xyz=-3.25 -1. 0. rpy=0 0 0
- joint chair_3_joint: origin xyz=-3. 3. 0. rpy=0 0 0 -> xyz=-3.25 1. 0. rpy=0 0 0
- joint chair_4_joint: origin xyz=3. -3. 0. rpy=0 0 0 -> xyz=0 3. 0. rpy=0 0 0
- joint chair_5_joint: origin xyz=3. 0. 0. rpy=0 0 0 -> xyz=3.25 1. 0. rpy=0 0 0
- joint chair_6_joint: origin xyz=3. 3. 0. rpy=0 0 0 -> xyz=3.25 -1. 0. rpy=0 0 0

File: mmseq_assets/scenes/xacro/restaurant.urdf.xacro (robot description, xacro)
@@ -54,20 +54,20 @@
   <link name="restaurant_base_link"/>
   <xacro:chair name="chair_1">
-    <origin rpy="0 0 0" xyz="-3. -3. 0."/>
+    <origin rpy="0 0 0" xyz="0 -3. 0."/>
   </xacro:chair>
   <xacro:chair name="chair_2">
-    <origin rpy="0 0 0" xyz="-3. 0. 0."/>
+    <origin rpy="0 0 0" xyz="-3.25 -1. 0."/>
   </xacro:chair>
   <xacro:chair name="chair_3">
-    <origin rpy="0 0 0" xyz="-3. 3. 0."/>
+    <origin rpy="0 0 0" xyz="-3.25 1. 0."/>
   </xacro:chair>
   <xacro:chair name="chair_4">
-    <origin rpy="0 0 0" xyz="3. -3. 0."/>
+    <origin rpy="0 0 0" xyz="0 3. 0."/>
   </xacro:chair>
   <xacro:chair name="chair_5">
-    <origin rpy="0 0 0" xyz="3. 0. 0."/>
+    <origin rpy="0 0 0" xyz="3.25 1. 0."/>
   </xacro:chair>
   <xacro:chair name="chair_6">
-    <origin rpy="0 0 0" xyz="3. 3. 0."/>
+    <origin rpy="0 0 0" xyz="3.25 -1. 0."/>
   </xacro:chair>
 </robot>

File: mmseq_assets/thing/xacro/collision.urdf.xacro (robot description, xacro)
@@ -49,5 +49,5 @@
     <child link="base_collision_link"/>
   </joint>
-  <xacro:collision_link_cylinder name="rack_collision_link" radius="0.275"/>
+  <xacro:collision_link_cylinder name="rack_collision_link" radius="0.325"/>
   <joint name="rack_collision_joint" type="fixed">
     <origin rpy="0 0 0" xyz="-0.45 -0. 0.75"/>
@@ -113,5 +113,5 @@
   </joint>
   <!-- Gripped Object -->
-  <xacro:collision_link_sphere name="gripped_object_collision_link" radius="0.22"/>
+  <xacro:collision_link_sphere name="gripped_object_collision_link" radius="0.26"/>
   <joint name="gripped_object_collision_joint" type="fixed">
     <origin rpy="0 0 0" xyz="0 0 0.0"/>
