Commit message: Updated link names in arm coverage urdf.

File: mmseq_assets/thing/xacro/arm_coverage.urdf.xacro (robot description, xacro)
@@ -10,5 +10,7 @@
           <sphere radius="${radius}"/>
         </geometry>
-        <material name="${material}"/>
+        <material name="coverage_ball_color">
+          <color rgba="1.0 0.0 0.0 0.0"/>
+        </material>
       </visual>
     </link>
@@ -27,27 +29,27 @@
     <child link="ur10_arm_forearm_coverage_link_1"/>
   </joint>
-  <xacro:coverage_link_sphere name="ur10_arm_forearm_coverage_sphere_link_2" radius="0.075"/>
+  <xacro:coverage_link_sphere name="ur10_arm_forearm_coverage_link_2" radius="0.075"/>
   <joint name="ur10_arm_forearm_coverage_sphere_joint_2" type="fixed">
     <origin rpy="0 1.5708 0" xyz="-0.275 0 0.06"/>
     <parent link="ur10_arm_forearm_link"/>
-    <child link="ur10_arm_forearm_coverage_sphere_link_2"/>
+    <child link="ur10_arm_forearm_coverage_link_2"/>
   </joint>
-  <xacro:coverage_link_sphere name="ur10_arm_forearm_coverage_sphere_link_3" radius="0.075"/>
+  <xacro:coverage_link_sphere name="ur10_arm_forearm_coverage_link_3" radius="0.075"/>
   <joint name="ur10_arm_forearm_coverage_sphere_joint_3" type="fixed">
     <origin rpy="0 1.5708 0" xyz="-0.35 0 0.06"/>
     <parent link="ur10_arm_forearm_link"/>
-    <child link="ur10_arm_forearm_coverage_sphere_link_3"/>
+    <child link="ur10_arm_forearm_coverage_link_3"/>
   </joint>
-  <xacro:coverage_link_sphere name="ur10_arm_forearm_coverage_sphere_link_4" radius="0.075"/>
+  <xacro:coverage_link_sphere name="ur10_arm_forearm_coverage_link_4" radius="0.075"/>
   <joint name="ur10_arm_forearm_coverage_sphere_joint_4" type="fixed">
     <origin rpy="0 1.5708 0" xyz="-0.425 0 0.06"/>
     <parent link="ur10_arm_forearm_link"/>
-    <child link="ur10_arm_forearm_coverage_sphere_link_4"/>
+    <child link="ur10_arm_forearm_coverage_link_4"/>
   </joint>
-  <xacro:coverage_link_sphere name="ur10_arm_forearm_coverage_sphere_link_5" radius="0.075"/>
+  <xacro:coverage_link_sphere name="ur10_arm_forearm_coverage_link_5" radius="0.075"/>
   <joint name="ur10_arm_forearm_coverage_sphere_joint_5" type="fixed">
     <origin rpy="0 1.5708 0" xyz="-0.5 0 0.06"/>
     <parent link="ur10_arm_forearm_link"/>
-    <child link="ur10_arm_forearm_coverage_sphere_link_5"/>
+    <child link="ur10_arm_forearm_coverage_link_5"/>
   </joint>
   <!-- Coverage sphere for the wrist -->
