Commit message: added collision link to rack

File: mmseq_assets/thing/xacro/collision.urdf.xacro (robot description, xacro)
@@ -23,4 +23,23 @@
     </link>
   </xacro:macro>
+    <xacro:macro name="collision_link_cylinder" params="name radius">
+    <link name="${name}">
+      <xacro:if value="$(arg use_collision)">
+        <collision>
+          <origin rpy="0 0 0" xyz="0 0 0" />
+          <geometry>
+            <cylinder  radius="${radius}" length="1"/>
+          </geometry>
+        </collision>
+      </xacro:if>
+      <visual>
+        <origin rpy="0 0 0" xyz="0 0 0" />
+        <geometry>
+          <cylinder  radius="${radius}" length="1"/>
+        </geometry>
+        <material name="${material}"/>
+      </visual>
+    </link>
+  </xacro:macro>
   <!-- Collision sphere for the base -->
   <xacro:collision_link_sphere name="base_collision_link" radius="0.6"/>
@@ -29,4 +48,10 @@
     <parent link="base_link"/>
     <child link="base_collision_link"/>
+  </joint>
+  <xacro:collision_link_cylinder name="rack_collision_link" radius="0.275"/>
+  <joint name="rack_collision_joint" type="fixed">
+    <origin rpy="0 0 0" xyz="-0.45 -0. 0.75"/>
+    <parent link="base_link"/>
+    <child link="rack_collision_link"/>
   </joint>
   <!-- Collision sphere for the upper arm -->

Commit message: Change base collision sphers to two.

File: mmseq_assets/thing/xacro/collision.urdf.xacro (robot description, xacro)
@@ -43,9 +43,21 @@
   </xacro:macro>
   <!-- Collision sphere for the base -->
-  <xacro:collision_link_sphere name="base_collision_link" radius="0.45"/>
+  <!-- <xacro:collision_link_sphere name="base_collision_link" radius="0.45"/>
   <joint name="base_collision_joint" type="fixed">
     <origin rpy="0 0 0" xyz="0 0 -0.08"/>
     <parent link="base_link"/>
     <child link="base_collision_link"/>
+  </joint> -->
+  <xacro:collision_link_sphere name="base_collision_link_front" radius="0.40"/>
+  <joint name="base_collision_joint_front" type="fixed">
+    <origin rpy="0 0 0" xyz="0.35 0 -0.08"/>
+    <parent link="base_link"/>
+    <child link="base_collision_link_front"/>
+  </joint>
+  <xacro:collision_link_sphere name="base_collision_link_back" radius="0.40"/>
+  <joint name="base_collision_joint_back" type="fixed">
+    <origin rpy="0 0 0" xyz="-0.25 0 -0.08"/>
+    <parent link="base_link"/>
+    <child link="base_collision_link_back"/>
   </joint>
   <xacro:collision_link_cylinder name="rack_collision_link" radius="0.325"/>
